File: pcb/clock.sch (EAGLE design)
At the start: 89 parts, among them Q1 BC849SMD, Q10 BC847BSMD, Q11 BC849SMD, Q12 BC849SMD, Q13 BC849SMD, Q14 BC857BSMD, Q15 BC847BSMD, Q16 BC857BSMD, Q17 BC847BSMD, Q18 BC857BSMD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

Commit message: funkcni prototyp
Parts:
- added S1, S2: (no value), switch-omron:31-XX
Connections:
- new net BL: U$10.BL, U$11.BL, U$12.BL, U$13.BL, U$4.BL, U$9.BL
- new net BOT: U$10.BOTTOM, U$11.BOTTOM, U$12.BOTTOM, U$13.BOTTOM, U$4.BOTTOM, U$9.BOTTOM
- new net BR: U$10.BR, U$11.BR, U$12.BR, U$13.BR, U$4.BR, U$9.BR
- new net DOT: U$10.DOT, U$11.DOT, U$12.DOT, U$13.DOT, U$4.DOT, U$9.DOT
- new net FIL_P: U$10.FIL_P, U$11.FIL_P, U$12.FIL_P, U$13.FIL_P, U$4.FIL_P, U$9.FIL_P
- new net MID: U$10.MIDDLE, U$11.MIDDLE, U$12.MIDDLE, U$13.MIDDLE, U$4.MIDDLE, U$9.MIDDLE
- new net N$54: U$4.FIL_M
- new net N$63: U$9.FIL_M
- new net N$68: U$11.GRID_P
- new net N$69: U$11.FIL_M
- new net N$70: U$10.GRID_P
- new net N$71: U$10.FIL_M
- new net N$72: U$4.GRID_P
- new net N$73: U$9.GRID_P
- new net N$74: U$12.GRID_P
- new net N$76: U$12.FIL_M
- new net N$77: U$13.GRID_P
- new net N$79: U$13.FIL_M
- new net TL: U$10.TL, U$11.TL, U$12.TL, U$13.TL, U$4.TL, U$9.TL
- new net TOP: U$10.TOP, U$11.TOP, U$12.TOP, U$13.TOP, U$4.TOP, U$9.TOP
- new net TR: U$10.TR, U$11.TR, U$12.TR, U$13.TR, U$4.TR, U$9.TR
- net G: now also U$5.K_B
Other:
- moved on the sheet: 16MHZ, BAT, C1, C2, JP1, JP2, Q11, Q12, Q13, Q9, R17, R18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
